Commit message: Phase 2: ros2_control diff drive, spec-filled controller params, drive test

File: ros2_ws/src/jgb_rover_description/urdf/gazebo.xacro (robot description, xacro)
@@ -14,4 +14,17 @@
   <xacro:surface link="caster_front_link" mu="${sim.caster.mu}"/>
   <xacro:surface link="caster_rear_link" mu="${sim.caster.mu}"/>
+  <!-- ===================== ros2_control ===================== -->
+  <xacro:property name="controllers_file" value="$(arg controllers_file)"/>
+  <xacro:if value="${controllers_file != ''}">
+    <gazebo>
+      <plugin filename="libign_ros2_control-system.so" name="ign_ros2_control::IgnitionROS2ControlPlugin">
+        <parameters>${controllers_file}</parameters>
+        <ros>
+          <remapping>/diff_drive_controller/cmd_vel:=/cmd_vel</remapping>
+          <remapping>/diff_drive_controller/odom:=/wheel/odom</remapping>
+        </ros>
+      </plugin>
+    </gazebo>
+  </xacro:if>
   <!-- ===================== ground truth ===================== -->
   <!-- Pose/twist of the model frame (= base_footprint) in the world. Bridged to

File: ros2_ws/src/jgb_rover_description/urdf/jgb_rover.urdf.xacro (robot description, xacro)
@@ -11,5 +11,7 @@
   <xacro:arg name="inject_errors" default="false"/>
   <xacro:arg name="sim_gazebo" default="true"/>
+  <!-- rendered controllers yaml (see jgb_rover_control.spec_params); empty = no gz ros2_control plugin -->
   <xacro:arg name="controllers_file" default=""/>
+  <xacro:arg name="hardware_plugin" default="jgb_rover_hardware/JgbRoverSystem"/>
   <!-- ===================== data ===================== -->
   <xacro:property name="pkg" value="$(find jgb_rover_description)"/>
@@ -93,5 +95,12 @@
       <collision>
         <origin xyz="0 0 0" rpy="${pi/2} 0 0"/>
-        <geometry><cylinder radius="${wheel_r * r_scale}" length="${wheel_w}"/></geometry>
+        <geometry>
+          <xacro:if value="${sim.wheel.collision == 'sphere'}">
+            <sphere radius="${wheel_r * r_scale}"/>
+          </xacro:if>
+          <xacro:if value="${sim.wheel.collision == 'cylinder'}">
+            <cylinder radius="${wheel_r * r_scale}" length="${wheel_w}"/>
+          </xacro:if>
+        </geometry>
       </collision>
       <inertial>
@@ -106,7 +115,9 @@
       <parent link="base_link"/>
       <child link="${side}_wheel_link"/>
-      <!-- wheel centre is given in base_footprint; with r_scale < 1 the axle stays put and the
-           wheel simply rolls on a smaller radius (sub-mm tilt, negligible) -->
-      <origin xyz="${centre[0]} ${centre[1]} ${centre[2] - base_z}" rpy="0 0 0"/>
+      <!-- wheel centre is given in base_footprint. With r_scale < 1 (error injection) the axle is
+           lowered by the radius difference so the smaller wheel still touches the floor; otherwise
+           the body would rest on the other wheel + the two centre-line casters and the small
+           wheel would hang in the air. -->
+      <origin xyz="${centre[0]} ${centre[1]} ${centre[2] - base_z - wheel_r * (1 - r_scale)}" rpy="0 0 0"/>
       <axis xyz="${wheel_axis[0]} ${wheel_axis[1]} ${wheel_axis[2]}"/>
       <limit effort="${wheel_effort_limit}" velocity="${wheel_vel_limit}"/>
@@ -176,4 +187,6 @@
     <origin xyz="${cam_xyz[0]} ${cam_xyz[1]} 0" rpy="0 0 0"/>
   </joint>
+  <!-- ===================== ros2_control ===================== -->
+  <xacro:include filename="$(find jgb_rover_description)/urdf/ros2_control.xacro"/>
   <!-- ===================== simulation ===================== -->
   <xacro:if value="$(arg sim_gazebo)">

Commit message: Phase 3: IMU, bias calibration with ZUPT, EKF fusion, error injection, odometry evaluation

File: ros2_ws/src/jgb_rover_description/urdf/gazebo.xacro (robot description, xacro)
@@ -18,5 +18,5 @@
   <xacro:if value="${controllers_file != ''}">
     <gazebo>
-      <plugin filename="libign_ros2_control-system.so" name="ign_ros2_control::IgnitionROS2ControlPlugin">
+      <plugin filename="libgz_ros2_control-system.so" name="gz_ros2_control::GazeboSimROS2ControlPlugin">
         <parameters>${controllers_file}</parameters>
         <ros>
@@ -27,4 +27,38 @@
     </gazebo>
   </xacro:if>
+  <!-- ===================== IMU (MPU6050) ===================== -->
+  <!-- 6-axis, no magnetometer: orientation output disabled; downstream treats it as unknown.
+       Gyro bias: gz-sensors draws it once from N(bias_mean, bias_stddev) and gives it a random
+       sign per axis, so the startup calibration node has something real to remove. -->
+  <xacro:property name="imu_n" value="${spec.imu.sim_noise}"/>
+  <xacro:macro name="imu_noise" params="stddev bias_mean bias_stddev">
+    <noise type="gaussian">
+      <mean>0.0</mean>
+      <stddev>${stddev}</stddev>
+      <bias_mean>${bias_mean}</bias_mean>
+      <bias_stddev>${bias_stddev}</bias_stddev>
+    </noise>
+  </xacro:macro>
+  <gazebo reference="${spec.imu.frame}">
+    <sensor name="imu" type="imu">
+      <always_on>true</always_on>
+      <update_rate>${spec.imu.rate_hz}</update_rate>
+      <topic>imu/data_raw</topic>
+      <ignition_frame_id>${spec.imu.frame}</ignition_frame_id>
+      <imu>
+        <enable_orientation>false</enable_orientation>
+        <angular_velocity>
+          <x><xacro:imu_noise stddev="${imu_n.gyro_stddev}" bias_mean="${imu_n.gyro_bias_mean}" bias_stddev="${imu_n.gyro_bias_stddev}"/></x>
+          <y><xacro:imu_noise stddev="${imu_n.gyro_stddev}" bias_mean="${imu_n.gyro_bias_mean}" bias_stddev="${imu_n.gyro_bias_stddev}"/></y>
+          <z><xacro:imu_noise stddev="${imu_n.gyro_stddev}" bias_mean="${imu_n.gyro_bias_mean}" bias_stddev="${imu_n.gyro_bias_stddev}"/></z>
+        </angular_velocity>
+        <linear_acceleration>
+          <x><xacro:imu_noise stddev="${imu_n.accel_stddev}" bias_mean="0.0" bias_stddev="${imu_n.accel_bias_stddev}"/></x>
+          <y><xacro:imu_noise stddev="${imu_n.accel_stddev}" bias_mean="0.0" bias_stddev="${imu_n.accel_bias_stddev}"/></y>
+          <z><xacro:imu_noise stddev="${imu_n.accel_stddev}" bias_mean="0.0" bias_stddev="${imu_n.accel_bias_stddev}"/></z>
+        </linear_acceleration>
+      </imu>
+    </sensor>
+  </gazebo>
   <!-- ===================== ground truth ===================== -->
   <!-- Pose/twist of the model frame (= base_footprint) in the world. Bridged to

File: ros2_ws/src/jgb_rover_description/urdf/ros2_control.xacro (robot description, xacro)
@@ -17,5 +17,5 @@
     <hardware>
       <xacro:if value="$(arg sim_gazebo)">
-        <plugin>ign_ros2_control/IgnitionSystem</plugin>
+        <plugin>gz_ros2_control/GazeboSimSystem</plugin>
       </xacro:if>
       <xacro:unless value="$(arg sim_gazebo)">

Commit message: Phase 4: camera, visual floor scan, slam_toolbox mapping, ArUco check, map evaluation

File: ros2_ws/src/jgb_rover_description/urdf/gazebo.xacro (robot description, xacro)
@@ -61,4 +61,33 @@
     </sensor>
   </gazebo>
+  <!-- ===================== camera (USB webcam) ===================== -->
+  <!-- Gazebo cameras look along +X of their link: camera_link is x-forward (pitched down).
+       Images are stamped with camera_optical_frame, as v4l2_camera will do on the robot. -->
+  <xacro:property name="cam_sim" value="${spec.camera.sim}"/>
+  <gazebo reference="${spec.camera.frame}">
+    <sensor name="camera" type="camera">
+      <always_on>true</always_on>
+      <update_rate>${cam_sim.fps}</update_rate>
+      <topic>camera/image_raw</topic>
+      <ignition_frame_id>camera_optical_frame</ignition_frame_id>
+      <camera name="webcam">
+        <horizontal_fov>${cam_sim.horizontal_fov}</horizontal_fov>
+        <image>
+          <width>${cam_sim.width}</width>
+          <height>${cam_sim.height}</height>
+          <format>R8G8B8</format>
+        </image>
+        <clip>
+          <near>${cam_sim.clip[0]}</near>
+          <far>${cam_sim.clip[1]}</far>
+        </clip>
+        <noise>
+          <type>gaussian</type>
+          <mean>0.0</mean>
+          <stddev>${cam_sim.noise_stddev}</stddev>
+        </noise>
+      </camera>
+    </sensor>
+  </gazebo>
   <!-- ===================== ground truth ===================== -->
   <!-- Pose/twist of the model frame (= base_footprint) in the world. Bridged to

File: ros2_ws/src/jgb_rover_description/urdf/jgb_rover.urdf.xacro (robot description, xacro)
@@ -163,6 +163,7 @@
   <link name="${spec.camera.frame}">
     <visual>
-      <!-- webcam.stl is in base_footprint coordinates, modelled at mesh_cad_pitch -->
-      <origin xyz="${-cam_xyz[0]} ${-cam_xyz[1]} ${-cam_xyz[2]}" rpy="0 ${-sim.camera.mesh_cad_pitch} 0"/>
+      <!-- webcam.stl is in base_footprint coordinates, modelled at mesh_cad_pitch; moved back by
+           mesh_clearance so the simulated lens is not inside its own housing -->
+      <origin xyz="${-cam_xyz[0] - sim.camera.mesh_clearance} ${-cam_xyz[1]} ${-cam_xyz[2]}" rpy="0 ${-sim.camera.mesh_cad_pitch} 0"/>
       <geometry><mesh filename="${mesh_dir}/webcam.stl"/></geometry>
       <material name="webcam_material"><color rgba="0.05 0.05 0.05 1"/></material>
